File: i2c-moist-sensor.sch (KiCad schematic (older format))
At the start: 21 parts, among them IC1 ATTINY441-SSU, P1 CONN_02X03, X1 16MHz

Commit message: Migrate to KiCad v.5
Parts:
- C1, C2, C3, C4, C5, C6: symbol C -> device:C
- D1, D2: symbol DIODESCH -> device:D_Schottky_ALT
- D3: symbol LED-RESCUE-i2c-moist-sensor -> device:LED_ALT
- IC1: symbol ATTINY441-SSU -> atmel:ATTINY441-SSU
- P1: symbol CONN_02X03 -> Connector:Conn_02x03_Odd_Even; Distributor (none) -> ?; Manufacturer (none) -> ?; PartNo (none) -> ?
- R1, R2, R4, R5, R6, R7, R8, R9: symbol R -> device:R
- TH1: symbol THERMISTOR -> device:Thermistor
- X1: symbol CRYSTAL -> device:Crystal
Connections:
- wire segments 34 -> 44
Changed lines of the file:
@@
-EESchema Schematic File Version 2
-LIBS:i2c-moist-sensor-rescue
-LIBS:power
-LIBS:device
-LIBS:transistors
-LIBS:conn
-LIBS:linear
-LIBS:regul
-LIBS:74xx
-LIBS:cmos4000
-LIBS:adc-dac
-LIBS:memory
-LIBS:xilinx
-LIBS:special
-LIBS:microcontrollers
-LIBS:dsp
-LIBS:microchip
-LIBS:analog_switches
-LIBS:motorola
-LIBS:texas
-LIBS:intel
-LIBS:audio
-LIBS:interface
-LIBS:digital-audio
-LIBS:philips
-LIBS:display
-LIBS:cypress
-LIBS:siliconi
-LIBS:opto
-LIBS:atmel
-LIBS:contrib
-LIBS:valves
+EESchema Schematic File Version 4
 LIBS:i2c-moist-sensor-cache
 EELAYER 26 0
@@
 $EndDescr
 $Comp
-L CRYSTAL X1
+L device:Crystal X1
 U 1 1 54D213EA
 P 5700 2800
@@
 F 2 "Crystals:Crystal_HC49-SD_SMD" H 5700 2800 60  0001 C CNN
 F 3 "" H 5700 2800 60  0000 C CNN
-F 4 "MULTICOMP" H 5700 2800 60  0001 C CNN "Manufacturer"
-F 5 " MCRSD16000F183000RR" H 5700 2800 60  0001 C CNN "PartNo"
+F 4 " MCRSD16000F183000RR" H 5700 2800 60  0001 C CNN "PartNo"
+F 5 "MULTICOMP" H 5700 2800 60  0001 C CNN "Manufacturer"
 F 6 "Farnell/2395958" H 5700 2800 60  0001 C CNN "Distributor"
 	1    5700 2800
@@
 $EndComp
 $Comp
-L C C1
+L device:C C1
 U 1 1 54D21881
 P 5400 2950
@@
 $EndComp
 $Comp
-L C C2
+L device:C C2
 U 1 1 54D218DE
 P 6000 2950
@@
 $EndComp
 $Comp
-L GND #PWR01
+L power:GND #PWR01
 U 1 1 54D21A04
 P 5700 3100
@@
 F 2 "" H 5700 3100 60  0000 C CNN
 F 3 "" H 5700 3100 60  0000 C CNN
+F 4 "?" H 5700 3100 60  0001 C CNN "PartNo"
+F 5 "?" H 5700 3100 60  0001 C CNN "Manufacturer"
+F 6 "?" H 5700 3100 60  0001 C CNN "Distributor"
 	1    5700 3100
 	1    0    0    -1
 $EndComp
 $Comp
-L VCC #PWR02
+L power:VCC #PWR02
 U 1 1 54D21DD5
 P 1550 1700
@@
 $EndComp
 $Comp
-L GND #PWR03
+L power:GND #PWR03
 U 1 1 54D21DE7
 P 1550 2900
@@
 F 2 "" H 1550 2900 60  0000 C CNN
 F 3 "" H 1550 2900 60  0000 C CNN
+F 4 "?" H 1550 2900 60  0001 C CNN "PartNo"
+F 5 "?" H 1550 2900 60  0001 C CNN "Manufacturer"
+F 6 "?" H 1550 2900 60  0001 C CNN "Distributor"
 	1    1550 2900
 	1    0    0    -1
 $EndComp
 $Comp
-L C C3
+L device:C C3
 U 1 1 54D21E5C
 P 1550 1850
@@
 $EndComp
 $Comp
-L GND #PWR04
+L power:GND #PWR04
 U 1 1 54D21F25
 P 1550 2000
@@
 F 2 "" H 1550 2000 60  0000 C CNN
 F 3 "" H 1550 2000 60  0000 C CNN
+F 4 "?" H 1550 2000 60  0001 C CNN "PartNo"
+F 5 "?" H 1550 2000 60  0001 C CNN "Manufacturer"
+F 6 "?" H 1550 2000 60  0001 C CNN "Distributor"
 	1    1550 2000
 	1    0    0    -1
 $EndComp
 $Comp
-L DIODESCH D1
+L device:D_Schottky_ALT D1
 U 1 1 54D21FCD
 P 9100 2350
@@
 $EndComp
 $Comp
-L DIODESCH D2
+L device:D_Schottky_ALT D2
 U 1 1 54D22068
 P 9100 3800
@@
 $EndComp
 $Comp
-L R R4
+L device:R R4
 U 1 1 54D2209D
 P 8350 3050
@@
 $EndComp
 $Comp
-L R R5
+L device:R R5
 U 1 1 54D22174
 P 9300 2200
@@
 $EndComp
 $Comp
-L R R8
+L device:R R8
 U 1 1 54D221C8
 P 9600 3950
@@
 $EndComp
 $Comp
-L GND #PWR06
+L power:GND #PWR06
 U 1 1 54D2221D
 P 9300 4100
@@
 F 2 "" H 9300 4100 60  0000 C CNN
 F 3 "" H 9300 4100 60  0000 C CNN
+F 4 "?" H 9300 4100 60  0001 C CNN "PartNo"
+F 5 "?" H 9300 4100 60  0001 C CNN "Manufacturer"
+F 6 "?" H 9300 4100 60  0001 C CNN "Distributor"
 	1    9300 4100
 	1    0    0    -1
 $EndComp
 $Comp
-L C C4
+L device:C C4
 U 1 1 54D2222A
 P 9300 2500
@@
 $EndComp
 $Comp
-L GND #PWR07
+L power:GND #PWR07
 U 1 1 54D222DF
 P 9300 2650
@@
 F 2 "" H 9300 2650 60  0000 C CNN
 F 3 "" H 9300 2650 60  0000 C CNN
+F 4 "?" H 9300 2650 60  0001 C CNN "PartNo"
+F 5 "?" H 9300 2650 60  0001 C CNN "Manufacturer"
+F 6 "?" H 9300 2650 60  0001 C CNN "Distributor"
 	1    9300 2650
 	1    0    0    -1
 $EndComp
 $Comp
-L R R7
+L device:R R7
 U 1 1 54D222F8
 P 9600 2500
@@
 SENSE_LOW
 $Comp
-L C C5
+L device:C C5
 U 1 1 54D22484
 P 9300 3950
@@
 $EndComp
 $Comp
-L R R6
+L device:R R6
 U 1 1 54D2252C
 P 9300 3650
@@
 SENSOR_TRACK
 $Comp
-L GND #PWR09
+L power:GND #PWR09
 U 1 1 54D22F14
 P 4750 5750
@@
 $EndComp
 $Comp
-L R R1
+L device:R R1
 U 1 1 54DF19BF
 P 4650 2900
@@
 $EndComp
 $Comp
-L VCC #PWR010
+L power:VCC #PWR010
 U 1 1 54DF1CF6
 P 4800 2900
@@
 $EndComp
 $Comp
-L C C6
+L device:C C6
 U 1 1 54DF1D15
 P 4500 3050
@@
 $EndComp
 $Comp
-L GND #PWR011
+L power:GND #PWR011
 U 1 1 54DF1D84
 P 4500 3200
@@
 F 2 "" H 4500 3200 60  0000 C CNN
 F 3 "" H 4500 3200 60  0000 C CNN
+F 4 "?" H 4500 3200 60  0001 C CNN "PartNo"
+F 5 "?" H 4500 3200 60  0001 C CNN "Manufacturer"
+F 6 "?" H 4500 3200 60  0001 C CNN "Distributor"
 	1    4500 3200
 	1    0    0    -1
@@
 SENSE_LOW
 $Comp
-L THERMISTOR TH1
+L device:Thermistor TH1
 U 1 1 54E05F89
-P 7250 4550
-F 0 "TH1" V 7350 4600 50  0000 C CNN
-F 1 "NCP18XH103F03RB" V 7150 4550 50  0000 C BNN
-F 2 "Resistors_SMD:R_0603" H 7250 4550 60  0001 C CNN
-F 3 "" H 7250 4550 60  0000 C CNN
-F 4 "NCP18XH103F03RB" V 7250 4550 60  0001 C CNN "PartNo"
-F 5 "MURATA" V 7250 4550 60  0001 C CNN "Manufacturer"
-F 6 "Farnell/2456122" V 7250 4550 60  0001 C CNN "Distributor"
-	1    7250 4550
-	1    0    0    -1
-$EndComp
-$Comp
-L R R2
+P 7250 4500
+F 0 "TH1" V 7350 4550 50  0000 C CNN
+F 1 "NCP18XH103F03RB" V 7150 4500 50  0000 C BNN
+F 2 "Resistors_SMD:R_0603" H 7250 4500 60  0001 C CNN
+F 3 "" H 7250 4500 60  0000 C CNN
+F 4 "NCP18XH103F03RB" V 7250 4500 60  0001 C CNN "PartNo"
+F 5 "MURATA" V 7250 4500 60  0001 C CNN "Manufacturer"
+F 6 "Farnell/2456122" V 7250 4500 60  0001 C CNN "Distributor"
+	1    7250 4500
+	1    0    0    -1
+$EndComp
+$Comp
+L device:R R2
 U 1 1 54E06028
 P 7250 4150
@@
 $EndComp
 $Comp
-L GND #PWR012
+L power:GND #PWR012
 U 1 1 54E0608E
-P 7250 4800
-F 0 "#PWR012" H 7250 4550 60  0001 C CNN
-F 1 "GND" H 7250 4650 60  0000 C CNN
-F 2 "" H 7250 4800 60  0000 C CNN
-F 3 "" H 7250 4800 60  0000 C CNN
-	1    7250 4800
+P 7250 4700
+F 0 "#PWR012" H 7250 4450 60  0001 C CNN
+F 1 "GND" H 7250 4550 60  0000 C CNN
+F 2 "" H 7250 4700 60  0000 C CNN
+F 3 "" H 7250 4700 60  0000 C CNN
+F 4 "?" H 7250 4700 60  0001 C CNN "PartNo"
+F 5 "?" H 7250 4700 60  0001 C CNN "Manufacturer"
+F 6 "?" H 7250 4700 60  0001 C CNN "Distributor"
+	1    7250 4700
 	1    0    0    -1
 $EndComp
@@
 THERMISTOR
 $Comp
-L LED-RESCUE-i2c-moist-sensor D3
+L device:LED_ALT D3
 U 1 1 54E06E01
 P 5100 1550
@@
 F 2 "LEDs:LED-0603" H 5100 1550 60  0001 C CNN
 F 3 "" H 5100 1550 60  0000 C CNN
-F 4 "KINGBRIGHT" H 5100 1550 60  0001 C CNN "Manufacturer"
-F 5 "KP-1608SURCK" H 5100 1550 60  0001 C CNN "PartNo"
+F 4 "KP-1608SURCK" H 5100 1550 60  0001 C CNN "PartNo"
+F 5 "KINGBRIGHT" H 5100 1550 60  0001 C CNN "Manufacturer"
 F 6 "Farnell/2449786" H 5100 1550 60  0001 C CNN "Distributor"
 	1    5100 1550
@@
 $EndComp
 $Comp
-L R R9
+L device:R R9
 U 1 1 54E06FCA
 P 5450 1550
@@
 	3650 2700 5400 2700
 Wire Wire Line
-	5400 3100 6000 3100
+	5400 3100 5700 3100
 Connection ~ 5700 3100
 Wire Wire Line
-	9300 2350 10500 2350
+	9300 2350 9600 2350
 Wire Wire Line
 	9600 2650 9300 2650
@@
 	9300 4100 9600 4100
 Wire Wire Line
-	9300 3800 10500 3800
+	9300 3800 9600 3800
 Connection ~ 9600 3800
 Wire Wire Line
-	8900 2350 8900 3800
+	8900 2350 8900 3050
 Wire Wire Line
 	8500 3050 8900 3050
@@
 	3650 2000 4550 2000
 $Comp
-L CONN_02X03 P1
+L Connector:Conn_02x03_Odd_Even P1
 U 1 1 54E0D5F3
-P 4500 5650
-F 0 "P1" H 4500 5850 50  0000 C CNN
-F 1 "CONN_02X03" H 4500 5450 50  0000 C CNN
-F 2 "Pin_Headers:Pin_Header_Straight_2x03" H 4500 4450 60  0001 C CNN
-F 3 "" H 4500 4450 60  0000 C CNN
-	1    4500 5650
-	1    0    0    -1
-$EndComp
-$Comp
-L VCC #PWR014
+P 4450 5650
+F 0 "P1" H 4450 5850 50  0000 C CNN
+F 1 "CONN_02X03" H 4450 5450 50  0000 C CNN
+F 2 "Pin_Headers:Pin_Header_Straight_2x03" H 4450 4450 60  0001 C CNN
+F 3 "" H 4450 4450 60  0000 C CNN
+F 4 "?" H 4450 5650 60  0001 C CNN "PartNo"
+F 5 "?" H 4450 5650 60  0001 C CNN "Manufacturer"
+F 6 "?" H 4450 5650 60  0001 C CNN "Distributor"
+	1    4450 5650
+	1    0    0    -1
+$EndComp
+$Comp
+L power:VCC #PWR014
 U 1 1 54E0D755
 P 4750 5550
@@
 Text Label 5650 5650 2    60   ~ 0
 MOSI/SDA
-Wire Wire Line
-	4250 5550 3850 5550
-Text Label 3850 5550 0    60   ~ 0
+Text Label 3350 5550 0    60   ~ 0
 MISO/SENSE_HIGH
-Wire Wire Line
-	4250 5650 3850 5650
-Text Label 3850 5650 0    60   ~ 0
+Text Label 3350 5650 0    60   ~ 0
 SCK/SCL
-Wire Wire Line
-	4250 5750 3850 5750
-Text Label 3850 5750 0    60   ~ 0
+Text Label 3350 5750 0    60   ~ 0
 RESET
-Connection ~ 9300 2350
-Wire Wire Line
-	3650 1900 9750 1900
+Wire Wire Line
+	3650 1900 7250 1900
 Wire Wire Line
 	5600 1800 3650 1800
@@
 	3650 2200 4550 2200
 $Comp
-L ATTINY441-SSU IC1
+L atmel:ATTINY441-SSU IC1
 U 1 1 556E13D2
 P 2600 2300
@@
 Text Label 7250 1900 0    60   ~ 0
 POWER
+Wire Wire Line
+	5700 3100 6000 3100
+Wire Wire Line
+	9600 2350 10500 2350
+Wire Wire Line
+	9600 3800 10500 3800
+Wire Wire Line
+	8900 3050 8900 3800
+Wire Wire Line
+	9300 1900 9750 1900
+Wire Wire Line
+	7250 1900 9300 1900
+Wire Wire Line
+	5550 2800 5400 2800
+Connection ~ 5400 2800
+Wire Wire Line
+	5850 2800 6000 2800
+Connection ~ 6000 2800
+Wire Wire Line
+	3350 5550 4250 5550
+Wire Wire Line
+	3350 5650 4250 5650
+Wire Wire Line
+	3350 5750 4250 5750
+Wire Wire Line
+	5250 1550 5300 1550
+Wire Wire Line
+	4900 1550 4950 1550
 $EndSCHEMATC
